File: ext_station_pcb/Stacja_pogody_SD.kicad_pcb (KiCad board)
At the start: 2 copper layers, 34.6 x 17.6 mm, 12 parts, among them J1 Zasilanie, J2 Conn_02x03_Odd_Even, U1 NRF24L01_Breakout, U2 ATtiny414-SS, U3 BME280

Commit message: poprawa plytki wew i zew
Parts:
- added R2: 4k7, Resistor_SMD:R_0603_1608Metric, B.Cu at (126.5, 45.8)
- added R3: 4k7, Resistor_SMD:R_0603_1608Metric, B.Cu at (130.5, 45.6)
Connections:
- net /BME_SCK renamed /BME_SCL
- net /BME_SDI renamed /BME_SDA
Routing:
- net VCC: track 37.4 -> 54.8 mm
- net /BME_SDA: track 16.1 -> 18.9 mm
- net /BME_SCL: track 14.0 -> 16.0 mm

Commit message: skonczona plytka dla plytki zew
Parts:
- U3: footprint Package_LGA:Bosch_LGA-8_2.5x2.5mm_P0.65mm_ClockwisePinNumbering -> my_footprints:Bosch_LGA-8_2.5x2.5mm_P0.65mm_ClockwisePinNumbering
- moved U3 0.70 mm to (131.1, 36.7)
Routing:
- net GND: track 11.5 -> 15.0 mm, vias 10 -> 12
- net VCC: track 54.8 -> 55.8 mm
- net /BME_SCL: track 16.0 -> 17.0 mm
- net /NRF_MOSI: track 13.1 -> 12.5 mm
- net Net-(U2-PA7): track 3.13 -> 3.65 mm
