File: ext_station_pcb/Stacja_pogody_SD.kicad_sch (KiCad schematic)
At the start: 12 parts, among them J1 Zasilanie, J2 Conn_02x03_Odd_Even, U1 NRF24L01_Breakout, U2 ATtiny414-SS, U3 BME280

Commit message: poprawa plytki wew i zew
Parts:
- added R2, R3: 4k7, Resistor_SMD:R_0603_1608Metric, symbol Device:R_Small
Connections:
- net VCC: now also R2.2, R3.2
- net BME_SCK renamed BME_SCL
- net BME_SCL: now also R3.1
- net BME_SDI renamed BME_SDA
- net BME_SDA: now also R2.1
Other:
- moved on the sheet: C1, C2, C3, U3

Commit message: skonczona plytka dla plytki zew
Parts:
- U3: footprint Package_LGA:Bosch_LGA-8_2.5x2.5mm_P0.65mm_ClockwisePinNumbering -> my_footprints:Bosch_LGA-8_2.5x2.5mm_P0.65mm_ClockwisePinNumbering
Changed lines of the file:
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@@
 			)
 		)
-		(property "Footprint" "Package_LGA:Bosch_LGA-8_2.5x2.5mm_P0.65mm_ClockwisePinNumbering"
+		(property "Footprint" "my_footprints:Bosch_LGA-8_2.5x2.5mm_P0.65mm_ClockwisePinNumbering"
 			(at 220.98 87.63 0)
 			(effects

Commit message: photos of project
Other:
- note added: "2 AA batteries power supply"
- note removed: "Zasilanie 2 paluszki AA"
- moved on the sheet: D1, H1, J2, R1, R2, R3, U1, U2, U3
